File: PowerMeter/PowerMeter.kicad_pcb (KiCad board)
At the start: 2 copper layers, 49.5 x 25.5 mm, 29 parts, among them IC1 AD8307, J1 RF Input, J2 DVM, J3 9v, J4 Switch, J5 0-1 mA, U2 LM1117-5.0, U3 LM358

Commit message: Minor changes preparing for production
Parts:
- moved C4 11.7 mm to (170.1, 87.3), turned to 90 degrees
- moved R3 10.9 mm to (167.1, 86.5), turned to 0 degrees
- moved C5 10.7 mm to (175.8, 79.8), turned to 270 degrees
- moved C9 8.14 mm to (183.0, 85.0), turned to 0 degrees
- moved C6 7.62 mm to (164.1, 87.4), turned to 90 degrees
- moved R6 6.35 mm to (157.7, 97.7)
- moved C7 5.72 mm to (160.8, 79.9), turned to 270 degrees
- moved U1 2.54 mm to (180.8, 80.8), turned to 180 degrees
- moved C3 2.41 mm to (176.8, 89.4), turned to 90 degrees
- moved C8 2.18 mm to (160.6, 93.6), turned to 270 degrees
- moved R7 2.11 mm to (165.6, 99.3)
- moved C10 1.96 mm to (161.7, 99.3)
- moved C1 1.21 mm to (187.4, 78.9)
- moved U2 0.83 mm to (167.1, 81.5)
- moved L1 0.83 mm to (191.3, 78.9)
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- renumbered IC1 to U1
Routing:
- net Net-(C4-Pad2): track 37.2 -> 16.0 mm
- net Net-(C3-Pad2): track 15.2 -> 24.9 mm
- net Net-(C1-Pad1): track 3.95 -> 12.1 mm
- net +5V: track 12.2 -> 8.09 mm
- net Net-(J5-Pad1): track 6.90 -> 10.4 mm
- net Net-(R5-Pad1): track 18.7 -> 15.9 mm
- net Net-(C8-Pad2): track 21.7 -> 20.3 mm
- net Net-(C2-Pad1): track 5.09 -> 6.01 mm
- net Net-(C10-Pad2): track 17.0 -> 16.1 mm
- net GND: vias 15 -> 19
Other:
- board size 49.5 x 25.5 mm -> 49.8 x 25.5 mm
- board text added: "RF Power Meter 1.0 AC3DN"
- board text added: "RF Power Meter 1.0 by AC3DN from June 2001 QST article "Simple RF-Power Measurement" by W7ZOI & W7PUA"
- board text removed: "RF Power Meter 1.0 June 2001 QST AC3DN"

Commit message: Updated README status
Parts:
- J3: value 9v -> 9v Battery
- J5: value 0-1 mA -> 0-1 mA Meter
- moved C9 4.96 mm to (178.2, 83.9), turned to 270 degrees
- moved R4 3.06 mm to (171.7, 95.5)
- moved R5 2.72 mm to (171.7, 98.9)
- moved C5 2.35 mm to (178.2, 79.8)
- moved R6 1.78 mm to (157.7, 95.9), turned to 270 degrees
- moved U1 1.73 mm to (182.2, 81.8), turned to 90 degrees
- moved C10 1.14 mm to (162.7, 99.8)
- moved R7 0.93 mm to (166.5, 99.0)
- moved C3 0.71 mm to (176.9, 88.7)
Routing:
- net Net-(C1-Pad1): track 12.1 -> 7.46 mm
- net Net-(C4-Pad2): track 16.0 -> 20.3 mm
- net Net-(C3-Pad2): track 24.9 -> 20.7 mm
- net Net-(C9-Pad2): track 4.54 -> 2.32 mm
- net Net-(R5-Pad1): track 15.9 -> 17.7 mm
- net Net-(J5-Pad1): track 10.4 -> 8.82 mm
- net GND: vias 19 -> 22

Commit message: Changed R8 to 6.8K
Parts:
- R8: value 6R8 -> 6K8
- renumbered U1 to IC1
Changed lines of the file:
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@@
     (tags "SOIC 1.27")
     (attr smd)
-    (fp_text reference U1 (at 4.2545 0 180) (layer F.SilkS)
+    (fp_text reference IC1 (at 4.2545 0 180) (layer F.SilkS)
       (effects (font (size 1 1) (thickness 0.15)))
     )
@@
       (effects (font (size 1 1) (thickness 0.15)))
     )
-    (fp_text value 6R8 (at 0.05588 2.2733 270) (layer F.Fab)
-      (effects (font (size 1 1) (thickness 0.15)))
-    )
+    (fp_text value 6K8 (at 0.05588 2.2733 270) (layer F.Fab)
+      (effects (font (size 1 1) (thickness 0.15)))
+    )
