File: HeadlessVFO/HeadlessVFO.kicad_pcb (KiCad board)
At the start: 2 copper layers, 39 parts, among them J1 Header_8x1, U1 AD8008, U2 AD9851, X1 TCXO

Commit message: Almost finished PCB
Parts:
- moved R15 16.9 mm to (134.9, 39.4), turned to 180 degrees
- moved C2 14.4 mm to (164.8, 58.2)
- moved R4 14.4 mm to (164.8, 54.4)
- moved R3 14.4 mm to (164.8, 50.6)
- moved R18 13.6 mm to (161.4, 55.7)
- moved C3 13.6 mm to (150.6, 67.0), turned to 180 degrees
- moved U1 13.5 mm to (159.3, 50.5)
- moved C6 13.2 mm to (146.4, 67.0), turned to 0 degrees
- moved R6 12.6 mm to (147.2, 63.2), turned to 90 degrees
- moved C5 10.8 mm to (155.4, 62.2), turned to 90 degrees
- moved R2 10.5 mm to (156.3, 45.7), turned to 0 degrees
- moved R9 10.5 mm to (149.7, 63.1), turned to 270 degrees
- moved R8 10.4 mm to (156.6, 57.5)
- moved J1 10.2 mm to (145.8, 35.6)
- moved R19 9.36 mm to (158.0, 62.0), turned to 90 degrees
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Routing:
- net Vcc: track 0.00 -> 122.6 mm, vias 0 -> 5
- net DATA: track 0.00 -> 28.8 mm
- net GND: track 0.00 -> 26.6 mm, vias 0 -> 21
- net CLOCK: track 0.00 -> 20.8 mm
- net Net-(C12-Pad1): track 0.38 -> 20.0 mm
- net LOAD: track 0.00 -> 19.6 mm, vias 0 -> 2
- net RFout: track 0.00 -> 19.0 mm
- net Net-(C13-Pad1): track 0.14 -> 18.6 mm
- net Net-(R2-Pad1): track 0.00 -> 18.0 mm
- net Net-(R10-Pad1): track 0.00 -> 13.9 mm
- net Net-(R17-Pad2): track 0.00 -> 12.4 mm
- net Net-(R18-Pad1): track 0.00 -> 12.2 mm
- net Net-(C3-Pad1): track 0.00 -> 10.9 mm
- net Net-(R11-Pad2): track 0.00 -> 8.20 mm
- net Net-(C1-Pad2): track 0.09 -> 7.61 mm
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Other:
- board text added: "GND"
- board text added: "Headless VFO 1.0 AC3DN"
- board text added: "RF"
- board text added: "Vcc"
- board text added: "clock"
- board text added: "data"
- board text added: "load"

Commit message: Final changes before making board
Parts:
- added REF***: OSHW-Logo2_7.3x6mm_SilkScreen, Symbols:OSHW-Logo2_7.3x6mm_SilkScreen, B.Cu at (164.1, 36.8)
- added REF***: OSHW-Logo2_7.3x6mm_SilkScreen, Symbols:OSHW-Logo2_7.3x6mm_SilkScreen, F.Cu at (164.1, 36.9)
- moved J1 2.17 mm to (148.0, 35.8)
Routing:
- net RFout: track 19.0 -> 16.2 mm
- net LOAD: track 19.6 -> 20.4 mm
- net Vcc: track 122.6 -> 123.4 mm
- net DATA: track 28.8 -> 29.5 mm
- net CLOCK: track 20.8 -> 20.2 mm
- net GND: vias 21 -> 15
Other:
- board outline added: 43.6 x 37.5 mm
